File: eagle/GabozePocaioRound2.brd (EAGLE design)
At the start: 73 x 114.5 mm, 32 parts, among them J1 AUDIO_JACK_3.5MM_KIT, J2 SPKR, J3 Batt Conn, J4 ZX62-B-5PA, U1 LM4875

Commit message: Wed  1 May 2019 12:41:43 EDT - changed thermals
Parts:
- A, B: value CONDUCTIVE_BUTTON -> CONDUCTIVE_BUTTONCONDUCTIVE_BUTTON_THICK; device 32teeth - Conductive Buttons:CONDUCTIVE_BUTTON -> 32teeth - Conductive Buttons:CONDUCTIVE_BUTTON_THICK
- DOWN, LEFT, RIGHT, UP: value CONDUCTIVE_BUTTON -> CONDUCTIVE_BUTTONCONDUCTIVE_BUTTON_DIRECTIONAL_THICK; device 32teeth - Conductive Buttons:CONDUCTIVE_BUTTON -> 32teeth - Conductive Buttons:CONDUCTIVE_BUTTON_DIRECTIONAL_THICK
- L1: value CONDUCTIVE_BUTTON_DRILL -> CONDUCTIVE_BUTTON_DRILLCONDUCTIVE_BUTTON_DRILL_THICK; device ConductiveButtons:CONDUCTIVE_BUTTON_DRILL -> 32teeth - Conductive Buttons:CONDUCTIVE_BUTTON_THICK_DRILL
- R1, X, Y: value CONDUCTIVE_BUTTON_DRILL -> CONDUCTIVE_BUTTON_DRILLCONDUCTIVE_BUTTON_DRILL_THICK; device 32teeth - Conductive Buttons:CONDUCTIVE_BUTTON_DRILL -> 32teeth - Conductive Buttons:CONDUCTIVE_BUTTON_THICK_DRILL
- SELECT, START: value CONDUCTIVE_BUTTON_STARTSELECT -> CONDUCTIVE_BUTTON_STARTSELECTCONDUCTIVE_BUTTON_THICK_STARTSELECT; device 32teeth - Conductive Buttons:CONDUCTIVE_BUTTON_STARTSELECT -> 32teeth - Conductive Buttons:CONDUCTIVE_BUTTON_THICK_STARTSELECT
- turned A to 90 degrees
- turned B to 90 degrees
- turned L1 to 90 degrees
- turned R1 to 90 degrees
- turned RIGHT to 180 degrees
- turned UP to 270 degrees
- turned X to 90 degrees
- turned Y to 90 degrees
Connections:
- net GND: now also SELECT.P$GND1, SELECT.P$GND2, SELECT.P$GND3, START.P$GND1, START.P$GND2, START.P$GND3
- net SELECT: now also SELECT.P$ACTIVE1, SELECT.P$ACTIVE2, SELECT.P$ACTIVE3
- net START: now also START.P$ACTIVE1, START.P$ACTIVE2, START.P$ACTIVE3
Routing:
- net RIGHT: track 57.0 -> 71.4 mm
- net X: track 44.9 -> 53.5 mm
- net A: track 64.9 -> 72.8 mm
- net R1: track 80.7 -> 86.5 mm
- net UP: track 59.1 -> 56.5 mm
- net B: track 74.9 -> 76.9 mm
- net Y: track 60.9 -> 62.5 mm
- net L1: track 79.5 -> 81.1 mm
- net START: track 101.4 -> 103.0 mm
- net LEFT: track 66.3 -> 67.7 mm
- net DOWN: track 80.2 -> 78.8 mm

Commit message: Correct the value of C2 to 220nF in Eagle and BOM files
In the datasheet of LM4875 [1], Texas Instruments recommends
a 0.22uF (which is 220nF [2]) AC-coupling capacitor at the
audio input port [3]. However, in the Eagle and BOM files of
Gaboze Pocaio Round 2, the capacitor value was specified
as 220pF by accident. Experiments showed that using a 220pF
capacitor instead of 220nF causes an audible distortion
of the headphone output, which is characterized by the lack
of bass due to the RC high-pass filter action.

This commit corrects the component value C2 from 220pF to
220nF in Eagle schematic and board design files. Also, in
the BOM,

    C2,CAP CER 220PF 50V X7R 0805,C0805C221M5RACTU

has been replaced by

    C2,CAP CER 0.22UF 50V X7R 0805,C0805C224K5RACTU

Applying this fix to the circuit board fixes the audible
distortion and allows the audio quality to be restored
to TI's reference design.

It should be note that the Gerber files are not corrected,
since the committer doesn't have the project settings required
to create an identical set of Gerber files. The Gerber files
should be updated in a later commit by the original author.

[1] https://www.ti.com/lit/ds/symlink/lm4875.pdf

[2] https://en.wikipedia.org/wiki/Metric_prefix

[3] See Figure 1.

Signed-off-by: Tom Li <tomli@tomli.me>
Parts:
- C2: value 220pF -> 220nF
Other:
- board text added: "100K 150 100uF 220nF 1uF 1uF"
- board text removed: "100K 150 100uF 220pF 1uF 1uF"
Changed lines of the file:
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@@
 150
 100uF
-220pF
+220nF
 1uF
 1uF</text>
@@
 </element>
 <element name="U1" library="texas" library_urn="urn:adsk.eagle:library:387" package="SOIC8" value="LM4875" x="12" y="6.5" smashed="yes" rot="MR90"/>
-<element name="C2" library="adafruit" library_urn="urn:adsk.eagle:library:420" package="C0805" value="220pF" x="5" y="8" smashed="yes" rot="MR0"/>
+<element name="C2" library="adafruit" library_urn="urn:adsk.eagle:library:420" package="C0805" value="220nF" x="5" y="8" smashed="yes" rot="MR0"/>
 <element name="C3" library="adafruit" library_urn="urn:adsk.eagle:library:420" package="C0805" value="1uF" x="22" y="5" smashed="yes" rot="MR180"/>
 <element name="C4" library="adafruit" library_urn="urn:adsk.eagle:library:420" package="C0805" value="1uF" x="5" y="5" smashed="yes" rot="MR0"/>
